Commit message: bicycle model controller iginition is added

File: bicycle_controller_ign/src/ign_ros2_control_demos/urdf/test_ackermann_drive.xacro.urdf (robot description, URDF)
Before this commit: robot ackermann_drive, 8 links, 7 joints
Links:
- removed link front_left_wheel_link
- removed link front_right_wheel_link
- removed link front_steer_left_link
- removed link front_steer_right_link
- removed link rear_left_link
- removed link rear_right_link
- added link front_steer_link, mass 0.5; collision box size=0.01 0.01 0.01; visual box size=0.01 0.01 0.01
- added link front_wheel_link, mass 1; collision cylinder length=0.14 radius=0.165; visual mesh filename=file://$(find ign_ros2_control_demos)/meshes/front_left_whe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
- added link rear_link, mass 1; collision cylinder length=0.14 radius=0.165; visual mesh filename=file://$(find ign_ros2_control_demos)/meshes/left_rear_link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
- link chassis: mass 10 -> 21
Joints:
- removed joint front_left_wheel_joint
- removed joint front_right_wheel_joint
- removed joint front_steer_left_joint
- removed joint front_steer_right_joint
- removed joint rear_left_joint
- removed joint rear_right_joint
- added joint front_steer_joint: type revolute, parent chassis, child front_steer_link, origin xyz=0.37142 0.0 -0.1955 rpy=1.5708 0 0, axis 0 1 0, limit lower=-100.57 upper=100.57 effort=1000.0 velocity=30
- added joint front_wheel_joint: type continuous, parent front_steer_link, child front_wheel_link, origin xyz=0 0 0 rpy=0 0 0, axis 0 0 1
- added joint rear_joint: type continuous, parent chassis, child rear_link, origin xyz=-0.28018 0 -0.1955 rpy=1.5708 0 0, axis 0 0 -1

Commit message: imu localization set up and bugs fixed

File: bicycle_controller_ign/src/ign_ros2_control_demos/urdf/test_ackermann_drive.xacro.urdf (robot description, URDF)
Before this commit: robot ackermann_drive, 6 links, 5 joints
Joints:
- joint chassis_joint: origin xyz=0.0266989327622036 0.000409203500587652 0.4 rpy=0 0 0 -> xyz=0.28018 0.0 0.4 rpy=0 0 0
