Commit message: model updated

File: acker_controller_ign/src/ign_ros2_control_demos/urdf/test_ackermann_drive.xacro.urdf (robot description, URDF)
Before this commit: robot ackermann_drive, 8 links, 7 joints
Links:
- removed link base_link
- removed link chassis
- removed link front_left_wheel_link
- removed link front_right_wheel_link
- removed link front_steer_left_link
- removed link front_steer_right_link
- removed link rear_left_link
- removed link rear_right_link
- added link front_left_strut, mass ${strut_mas}; collision box size=${strut_wid} ${strut_wid} ${strut_wid}; visual box size=${strut_wid} ${strut_wid} ${strut_wid}
- added link front_left_wheel, mass ${wheel_mas}; collision cylinder length=${wheel_wid} radius=${wheel_rad}; visual mesh filename=file://$(find ign_ros2_control_demos)/meshes/front_left_whe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
- added link front_right_strut, mass ${strut_mas}; collision box size=${strut_wid} ${strut_wid} ${strut_wid}; visual box size=${strut_wid} ${strut_wid} ${strut_wid}
- added link front_right_wheel, mass ${wheel_mas}; collision cylinder length=${wheel_wid} radius=${wheel_rad}; visual mesh filename=file://$(find ign_ros2_control_demos)/meshes/front_left_whe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
- added link imu_link, mass 0.1; collision box size=0.1 0.1 0.1; visual box size=0.1 0.1 0.1
- added link rear_left_strut, mass ${strut_mas}; collision box size=${strut_wid} ${strut_wid} ${strut_wid}; visual box size=${strut_wid} ${strut_wid} ${strut_wid}
- added link rear_left_wheel, mass ${wheel_mas}; collision cylinder length=${wheel_wid} radius=${wheel_rad}; visual mesh filename=file://$(find ign_ros2_control_demos)/meshes/left_rear_link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
- added link rear_right_strut, mass ${strut_mas}; collision box size=${strut_wid} ${strut_wid} ${strut_wid}; visual box size=${strut_wid} ${strut_wid} ${strut_wid}
- added link rear_right_wheel, mass ${wheel_mas}; collision cylinder length=${wheel_wid} radius=${wheel_rad}; visual mesh filename=file://$(find ign_ros2_control_demos)/meshes/left_rear_link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
- added link steerbot_chassis, mass ${chassis_mas}; collision mesh filename=file://$(find ign_ros2_control_demos)/meshes/base_link.STL; visual mesh filename=file://$(find ign_ros2_control_demos)/meshes/base_link.STL
- added link steerbot_footprint
Joints:
- removed joint chassis_joint
- removed joint front_left_wheel_joint
- removed joint front_right_wheel_joint
- removed joint front_steer_left_joint
- removed joint front_steer_right_joint
- removed joint rear_left_joint
- removed joint rear_right_joint
- added joint front_left_steer_bearing: type continuous, parent steerbot_chassis, child front_left_strut, origin xyz=0.37142 0.3025 -0.1955 rpy=0 0 0, axis 0 0 1, limit effort=1000 velocity=1000
- added joint front_left_wheel_bearing: type continuous, parent front_left_strut, child front_left_wheel, origin xyz=0 ${strut_wid+.002} 0 rpy=0 0 0, axis 0 1 0, limit effort=1000 velocity=1000
- added joint front_right_steer_bearing: type continuous, parent steerbot_chassis, child front_right_strut, origin xyz=0.37142 -0.3025 -0.1955 rpy=0 0 0, axis 0 0 1, limit effort=1000 velocity=1000
- added joint front_right_wheel_bearing: type continuous, parent front_right_strut, child front_right_wheel, origin xyz=0 -${strut_wid+.002} 0 rpy=0 0 0, axis 0 1 0, limit effort=1000 velocity=1000
- added joint imu_joint: type fixed, parent steerbot_chassis, child imu_link, origin xyz=-0.28018 0 0 rpy=0 0 0
- added joint rear_left_steer_bearing: type fixed, parent steerbot_chassis, child rear_left_strut, origin xyz=-0.28018 0.3025 -0.19558 rpy=0 0 0, axis 0 0 1, limit effort=1000 velocity=1000
- added joint rear_left_wheel_bearing: type continuous, parent rear_left_strut, child rear_left_wheel, origin xyz=0 ${strut_wid+.002} 0 rpy=0 0 0, axis 0 1 0, limit effort=1000 velocity=1000
- added joint rear_right_steer_bearing: type fixed, parent steerbot_chassis, child rear_right_strut, origin xyz=-0.28018 -0.3025 -0.19558 rpy=0 0 0, axis 0 0 1, limit effort=1000 velocity=1000
- added joint rear_right_wheel_bearing: type continuous, parent rear_right_strut, child rear_right_wheel, origin xyz=0 -${strut_wid+.002} 0 rpy=0 0 0, axis 0 1 0, limit effort=1000 velocity=1000
- added joint steerbot_footprint_joint: type fixed, parent steerbot_footprint, child steerbot_chassis, origin xyz=0.28018 0 1.0 rpy=0 0 0

Commit message: ackermann simulation tested

File: acker_controller_ign/src/ign_ros2_control_demos/urdf/test_ackermann_drive.xacro.urdf (robot description, URDF)
Before this commit: robot ackermann_drive, 11 links, 10 joints
Links:
- added link SK_link, mass 3; collision mesh filename=file://$(find ign_ros2_control_demos)/meshes/SK_link.STL; visual mesh filename=file://$(find ign_ros2_control_demos)/meshes/SK_link.STL
- added link camera_link, mass 0.2; collision mesh filename=file://$(find ign_ros2_control_demos)/meshes/camera_link.STL; visual mesh filename=file://$(find ign_ros2_control_demos)/meshes/camera_link.STL
- added link lidar_link, mass 0.8; collision mesh filename=file://$(find ign_ros2_control_demos)/meshes/lidar_link.STL; visual mesh filename=file://$(find ign_ros2_control_demos)/meshes/lidar_link.STL
- link imu_link: mass 0.1 -> 0.011717; geometry collision mesh filename=file://$(find ign_ros2_control_demos)/meshes/imu_link.STL; visual mesh filename=file://$(find ign_ros2_control_demos)/meshes/imu_link.STL
Joints:
- added joint camera_joint: type fixed, parent SK_link, child camera_link, origin xyz=0 0 0 rpy=0 0 0
- added joint lidar_joint: type fixed, parent SK_link, child lidar_link, origin xyz=0 0 0 rpy=0 0 0
- added joint sensor_kit_base_joint: type fixed, parent steerbot_chassis, child SK_link, origin xyz=0.4225 0.0 0.016 rpy=0 0 0
- joint imu_joint: origin xyz=-0.28018 0 0 rpy=0 0 0 -> xyz=0 0 0 rpy=0 0 0; parent steerbot_chassis -> SK_link
